Commit message: Update cybergear models

File: cybergear_description/urdf/cybergear.urdf.xacro (robot description, xacro)
@@ -1,48 +1,50 @@
 <?xml version="1.0"?>
 <robot name="cybergear" xmlns:xacro="http://www.ros.org/wiki/xacro" >
-  <link name="body">
-    <visual>
+  <xacro:macro name="cybergear" params="prefix">
+    <link name="${prefix}outer_body">
+      <visual>
+        <origin xyz="0 0 0" rpy="0 0 0"/>
+        <geometry>
+          <mesh filename="package://cybergear_description/meshes/cybergear_outer_body.stl"/>
+        </geometry>
+        <material name="gray">
+          <color rgba="0.8 0.8 0.8 1.0"/>
+        </material>
+      </visual>
+    </link>
+    <link name="${prefix}inner_body">
+      <visual>
+        <origin xyz="0 0 0" rpy="0 0 0"/>
+        <geometry>
+          <mesh filename="package://cybergear_description/meshes/cybergear_inner_body.stl"/>
+        </geometry>
+        <material name="gray">
+          <color rgba="0.8 0.8 0.8 1.0"/>
+        </material>
+      </visual>
+    </link>
+    <link name="${prefix}arm">
+      <visual>
+        <origin xyz="0 0 0" rpy="0 0 0"/>
+        <geometry>
+          <mesh filename="package://cybergear_description/meshes/arm110.stl"/>
+        </geometry>
+        <material name="gray">
+          <color rgba="0.8 0.8 0.8 1.0"/>
+        </material>
+      </visual>
+    </link>
+    <joint name="${prefix}joint" type="revolute">
       <origin xyz="0 0 0" rpy="0 0 0"/>
-      <geometry>
-        <mesh filename="package://cybergear_description/meshes/cybergear_outer_body.stl"/>
-      </geometry>
-      <material name="gray">
-        <color rgba="0.8 0.8 0.8 1.0"/>
-      </material>
-    </visual>
-  </link>
-  <link name="inner_body">
-    <visual>
+      <axis xyz="1 0 0"/>
+      <parent link="${prefix}outer_body"/>
+      <child link="${prefix}inner_body"/>
+      <limit lower="-1.5" upper="1.5" effort="0" velocity="0"/>
+    </joint>
+    <joint name="${prefix}inner_body_arm_joint" type="fixed">
       <origin xyz="0 0 0" rpy="0 0 0"/>
-      <geometry>
-        <mesh filename="package://cybergear_description/meshes/cybergear_inner_body.stl"/>
-      </geometry>
-      <material name="gray">
-        <color rgba="0.8 0.8 0.8 1.0"/>
-      </material>
-    </visual>
-  </link>
-  <link name="arm">
-    <visual>
-      <origin xyz="0 0 0" rpy="0 0 0"/>
-      <geometry>
-        <mesh filename="package://cybergear_description/meshes/arm110.stl"/>
-      </geometry>
-      <material name="gray">
-        <color rgba="0.8 0.8 0.8 1.0"/>
-      </material>
-    </visual>
-  </link>
-  <joint name="motor_joint" type="revolute">
-    <origin xyz="0 0 0" rpy="0 0 0"/>
-    <axis xyz="1 0 0"/>
-    <parent link="body"/>
-    <child link="inner_body"/>
-    <limit lower="-1.5" upper="1.5" effort="0" velocity="0"/>
-  </joint>
-  <joint name="inner_body_arm_joint" type="fixed">
-    <origin xyz="0 0 0" rpy="0.0 0.0 0.0"/>
-    <parent link="inner_body"/>
-    <child link="arm"/>
-  </joint>
+      <parent link="${prefix}inner_body"/>
+      <child link="${prefix}arm"/>
+    </joint>
+  </xacro:macro>
 </robot>

File: cybergear_description/urdf/cybergear_1dof.urdf.xacro (robot description, xacro)
@@ -3,15 +3,8 @@
   <xacro:include filename="$(find cybergear_description)/urdf/cybergear.urdf.xacro"/>
   <xacro:cybergear prefix="motor1_"/>
-  <xacro:cybergear prefix="motor2_"/>
   <link name="origin"/>
-  <joint name="origin_to_motor1" type="fixed">
-    <origin xyz="-0.1 0 0" rpy="${pi} 0 ${-pi/2}"/>
+  <joint name="origin_to_cybergear" type="fixed">
     <parent link="origin"/>
     <child link="motor1_outer_body"/>
   </joint>
-  <joint name="origin_to_motor2" type="fixed">
-    <origin xyz="0.1 0 0" rpy="${pi} 0 ${-pi/2}"/>
-    <parent link="origin"/>
-    <child link="motor2_outer_body"/>
-  </joint>
 </robot>
